Commit message: Added meshes. Added S1

File: robomaster_description/urdf/arm.urdf.xacro (robot description, xacro)
@@ -1,6 +1,6 @@
 <?xml version="1.0"?>
 <robot xmlns:xacro="http://playerstage.sourceforge.net/gazebo/xmlschema/#xacro">
-  <xacro:macro name="arm">
-    <link name="arm_1_link">
+  <xacro:macro name="arm" params="tf_prefix=''">
+    <link name="${tf_prefix}arm_1_link">
       <inertial>
         <origin xyz="-0.0005586 0.023592 0.0011729" rpy="0 0 0"/>
@@ -31,5 +31,5 @@
     <!-- <link name="arm_2_dummy">
     </link> -->
-    <link name="arm_2_link">
+    <link name="${tf_prefix}arm_2_link">
       <inertial>
         <origin xyz="0.0222614 -0.0202749 -0.008504" rpy="0 0 0"/>
@@ -75,5 +75,5 @@
       </inertial>
     </link> -->
-    <link name="arm_base_link">
+    <link name="${tf_prefix}arm_base_link">
       <inertial>
         <origin xyz="0 0 0" rpy="0 0 0"/>
@@ -109,7 +109,7 @@
       </collision>
     </link>
-    <link name="end_point_link">
-    </link>
-    <link name="endpoint_bracket_link">
+    <link name="${tf_prefix}end_point_link">
+    </link>
+    <link name="${tf_prefix}endpoint_bracket_link">
       <inertial>
         <origin xyz="0.0116468 -0.0288044 0.0041342" rpy="0 0 0"/>
@@ -133,5 +133,5 @@
     <!-- <link name="rod_1_dummy">
     </link> -->
-    <link name="rod_1_link">
+    <link name="${tf_prefix}rod_1_link">
       <inertial>
         <origin xyz="-0.0477809 0 0.0272644" rpy="0 0 0"/>
@@ -160,5 +160,5 @@
       </inertial>
     </link> -->
-    <link name="rod_2_link">
+    <link name="${tf_prefix}rod_2_link">
       <inertial>
         <origin xyz="0.0011528 0 0.0549123" rpy="0 0 0"/>
@@ -187,5 +187,5 @@
       </inertial>
     </link> -->
-    <link name="rod_3_link">
+    <link name="${tf_prefix}rod_3_link">
       <inertial>
         <origin xyz="-0.0003574 9.5e-06 0.0001674" rpy="0 0 0"/>
@@ -207,5 +207,5 @@
       </collision>
     </link>
-    <link name="rod_link">
+    <link name="${tf_prefix}rod_link">
       <inertial>
         <origin xyz="-8.11e-05 0.0023793 8.58e-05" rpy="0 0 0"/>
@@ -236,5 +236,5 @@
     <!-- <link name="triangle_2_dummy">
     </link> -->
-    <link name="triangle_link">
+    <link name="${tf_prefix}triangle_link">
       <inertial>
         <origin xyz="0.1417841 0.0321051 -0.1257179" rpy="0 0 0"/>
@@ -256,8 +256,8 @@
       </collision>
     </link>
-    <joint name="arm_1_joint" type="revolute">
+    <joint name="${tf_prefix}arm_1_joint" type="revolute">
       <origin xyz="0.0103961 -0.0255713 0.030741" rpy="0 0 0"/>
-      <parent link="arm_base_link"/>
-      <child link="arm_1_link"/>
+      <parent link="${tf_prefix}arm_base_link"/>
+      <child link="${tf_prefix}arm_1_link"/>
       <axis xyz="0.0 1.0 0"/>
       <limit effort="0" velocity="0" lower="-0.274" upper="1.384"/>
@@ -268,11 +268,11 @@
       <child link="arm_2_dummy"/>
     </joint> -->
-    <joint name="arm_2_joint" type="continuous">
+    <joint name="${tf_prefix}arm_2_joint" type="continuous">
       <origin xyz="0.0018704 0.0438659 0.1210238" rpy="0 0 0"/>
-      <parent link="arm_1_link"/>
-      <child link="arm_2_link"/>
+      <parent link="${tf_prefix}arm_1_link"/>
+      <child link="${tf_prefix}arm_2_link"/>
       <axis xyz="0.0 1.0 0"/>
       <limit effort="0" velocity="0"/>
-      <mimic joint="rod_3_joint" multiplier="-1.0" offset="0.0"/>
+      <mimic joint="${tf_prefix}rod_3_joint" multiplier="-1.0" offset="0.0"/>
     </joint>
     <!-- <joint name="arm_base_attachment_joint" type="fixed">
@@ -281,8 +281,8 @@
       <child link="arm_base_attachment_link"/>
     </joint> -->
-    <joint name="arm_base_joint" type="fixed">
+    <joint name="${tf_prefix}arm_base_joint" type="fixed">
       <origin xyz="0 0.0010384 0.0906477" rpy="0 0 0"/>
-      <parent link="chassis_base_link"/>
-      <child link="arm_base_link"/>
+      <parent link="${tf_prefix}chassis_base_link"/>
+      <child link="${tf_prefix}arm_base_link"/>
     </joint>
     <!-- <joint name="attachement_link" type="floating">
@@ -291,15 +291,15 @@
       <child link="attachement_link"/>
     </joint> -->
-    <joint name="end_point_joint" type="fixed">
+    <joint name="${tf_prefix}end_point_joint" type="fixed">
       <origin xyz="0.0110125 -0.0270264 -0.0103816" rpy="0 0 0"/>
-      <parent link="endpoint_bracket_link"/>
-      <child link="end_point_link"/>
-    </joint>
-    <joint name="endpoint_bracket_joint" type="continuous">
+      <parent link="${tf_prefix}endpoint_bracket_link"/>
+      <child link="${tf_prefix}end_point_link"/>
+    </joint>
+    <joint name="${tf_prefix}endpoint_bracket_joint" type="continuous">
       <origin xyz="0.1058557 0.006752 -0.0561093" rpy="0 0 0"/>
-      <parent link="arm_2_link"/>
-      <child link="endpoint_bracket_link"/>
-      <axis xyz="0.0 1.0 0"/>
-      <mimic joint="rod_joint" multiplier="-1.0" offset="0.0"/>
+      <parent link="${tf_prefix}arm_2_link"/>
+      <child link="${tf_prefix}endpoint_bracket_link"/>
+      <axis xyz="0.0 1.0 0"/>
+      <mimic joint="${tf_prefix}rod_joint" multiplier="-1.0" offset="0.0"/>
       <!-- <limit effort="0" velocity="0"/> -->
     </joint>
@@ -309,10 +309,10 @@
       <child link="rod_1_dummy"/>
     </joint> -->
-    <joint name="rod_1_joint" type="continuous">
+    <joint name="${tf_prefix}rod_1_joint" type="continuous">
       <origin xyz="0.0134583 -0.0540971 0.0213068" rpy="0 -0.021293 0"/>
-      <parent link="endpoint_bracket_link"/>
-      <child link="rod_1_link"/>
-      <axis xyz="0.0 1.0 0"/>
-      <mimic joint="rod_joint" multiplier="1.0" offset="0.0"/>
+      <parent link="${tf_prefix}endpoint_bracket_link"/>
+      <child link="${tf_prefix}rod_1_link"/>
+      <axis xyz="0.0 1.0 0"/>
+      <mimic joint="${tf_prefix}rod_joint" multiplier="1.0" offset="0.0"/>
       <!-- <limit effort="0" velocity="0"/> -->
     </joint>
@@ -322,10 +322,10 @@
       <child link="rod_2_dummy"/>
     </joint> -->
-    <joint name="rod_2_joint" type="continuous">
+    <joint name="${tf_prefix}rod_2_joint" type="continuous">
       <origin xyz="-0.0224276 -0.0290701 0.0554782" rpy="0 -0.0094248 0"/>
-      <parent link="arm_base_link"/>
-      <child link="rod_2_link"/>
-      <axis xyz="0.0 1.0 0"/>
-      <mimic joint="arm_1_joint" multiplier="1.0" offset="0.0"/>
+      <parent link="${tf_prefix}arm_base_link"/>
+      <child link="${tf_prefix}rod_2_link"/>
+      <axis xyz="0.0 1.0 0"/>
+      <mimic joint="${tf_prefix}arm_1_joint" multiplier="1.0" offset="0.0"/>
       <!-- <limit effort="0" velocity="0"/> -->
     </joint>
@@ -335,15 +335,15 @@
       <child link="rod_3_dummy"/>
     </joint> -->
-    <joint name="rod_3_joint" type="revolute">
+    <joint name="${tf_prefix}rod_3_joint" type="revolute">
       <origin xyz="-0.042397 0.0004533 0.0223131" rpy="0 0 0"/>
-      <parent link="rod_link"/>
-      <child link="rod_3_link"/>
+      <parent link="${tf_prefix}rod_link"/>
+      <child link="${tf_prefix}rod_3_link"/>
       <axis xyz="0.0 1.0 0"/>
       <limit effort="0" velocity="0" lower="-0.34732" upper="1.21475"/>
     </joint>
-    <joint name="rod_joint" type="revolute">
+    <joint name="${tf_prefix}rod_joint" type="revolute">
       <origin xyz="0.009805 0.0214241 0.0319234" rpy="0 0 0"/>
-      <parent link="arm_base_link"/>
-      <child link="rod_link"/>
+      <parent link="${tf_prefix}arm_base_link"/>
+      <child link="${tf_prefix}rod_link"/>
       <axis xyz="0.0 1.0 0"/>
       <limit effort="0" velocity="0" lower="-0.79936" upper="1.73137"/>
@@ -359,10 +359,10 @@
       <child link="triangle_2_dummy"/>
     </joint> -->
-    <joint name="triangle_joint" type="continuous">
+    <joint name="${tf_prefix}triangle_joint" type="continuous">
       <origin xyz="0.0020224 -0.007103 0.1212334" rpy="0 0.2502802 0"/>
-      <parent link="arm_1_link"/>
-      <child link="triangle_link"/>
-      <axis xyz="0.0 1.0 0"/>
-      <mimic joint="arm_1_joint" multiplier="-1.0" offset="0.0"/>
+      <parent link="${tf_prefix}arm_1_link"/>
+      <child link="${tf_prefix}triangle_link"/>
+      <axis xyz="0.0 1.0 0"/>
+      <mimic joint="${tf_prefix}arm_1_joint" multiplier="-1.0" offset="0.0"/>
     </joint>
     </xacro:macro>

File: robomaster_description/urdf/base.urdf.xacro (robot description, xacro)
@@ -1,10 +1,9 @@
 <?xml version="1.0"?>
-  <robot xmlns:xacro="http://playerstage.sourceforge.net/gazebo/xmlschema/#xacro" name="robomaster_ep_base">
+  <robot xmlns:xacro="http://playerstage.sourceforge.net/gazebo/xmlschema/#xacro">
   <xacro:include filename="led.urdf.xacro"/>
   <xacro:include filename="wheel.urdf.xacro"/>
-  <xacro:include filename="intelligent_controller.urdf.xacro"/>
-  <xacro:macro name="robomaster_ep_base">
-    <link name="base_link"/>
-    <link name="chassis_base_link">
+  <xacro:macro name="base" params="tf_prefix=''">
+    <link name="${tf_prefix}base_link"/>
+    <link name="${tf_prefix}chassis_base_link">
       <inertial>
         <origin xyz="-0.0058789 -0.0001128 0.0294307" rpy="0 0 0"/>
@@ -68,50 +67,17 @@
       </collision>
     </link>
-    <joint name="chassis_base_joint" type="fixed">
+    <joint name="${tf_prefix}chassis_base_joint" type="fixed">
       <origin xyz="0 0 0.03465" rpy="0 0 0"/>
-      <parent link="base_link"/>
-      <child link="chassis_base_link"/>
+      <parent link="${tf_prefix}base_link"/>
+      <child link="${tf_prefix}chassis_base_link"/>
     </joint>
-    <link name="extension_base_link">
-      <inertial>
-        <origin xyz="0.0044194 -1.08e-05 0.00431" rpy="0 0 0"/>
-        <mass value="0.22"/>
-        <inertia ixx="0.00133" ixy="0" ixz="0" iyy="0.00092" iyz="0" izz="0.00224"/>
-      </inertial>
-      <visual name="extension_base">
-        <origin xyz="0 0 0" rpy="0 0 0"/>
-        <geometry>
-          <mesh filename="package://robomaster_description/meshes/extension_base.dae" scale="1.0 1.0 1.0"/>
-        </geometry>
-        <material name="metal"/>
-      </visual>
-      <visual name="extension_support">
-        <origin xyz="-0.078582 0.0075392 0.0046459" rpy="0 0 0"/>
-        <geometry>
-          <mesh filename="package://robomaster_description/meshes/extension_support.dae" scale="1.0 1.0 1.0"/>
-        </geometry>
-        <material name="metal"/>
-      </visual>
-      <collision name="ExtensionBase">
-        <origin xyz="0.0044194 -1.08e-05 0.00431" rpy="0 0 0"/>
-        <geometry>
-          <box size="0.2796935 0.2317787 0.013"/>
-        </geometry>
-      </collision>
-    </link>
-    <joint name="extension_base_joint" type="fixed">
-      <origin xyz="-0.0091948 0.0010492 0.070543" rpy="0 0 0"/>
-      <parent link="chassis_base_link"/>
-      <child link="extension_base_link"/>
-    </joint>
-    <xacro:chassis_module name="front" xyz="0.1569985 -0.0004276 0.0432862" rpy="0 0 0"/>
-    <xacro:chassis_module name="left" xyz="-0.0024413 0.0886932 0.0298341" rpy="0 0 ${pi/2}"/>
-    <xacro:chassis_module name="rear" xyz="-0.1581827 -0.0027864 0.0303668" rpy="0 0 ${pi}"/>
-    <xacro:chassis_module name="right" xyz="-0.0024413 -0.0886932 0.0298341" rpy="0 0 ${-pi/2}"/>
-    <xacro:wheel name="front_left" xyz="0.1 0.1 0.01535" direction="1" side="1"/>
-    <xacro:wheel name="front_right" xyz="0.1 -0.1 0.01535" direction="-1" side="-1"/>
-    <xacro:wheel name="rear_left" xyz="-0.1 0.1 0.01535" direction="-1" side="1"/>
-    <xacro:wheel name="rear_right" xyz="-0.1 -0.1 0.01535" direction="1" side="-1"/>
-    <xacro:intelligent_controller/>
+    <xacro:chassis_module tf_prefix="${tf_prefix}" name="front" xyz="0.1569985 -0.0004276 0.0432862" rpy="0 0 0"/>
+    <xacro:chassis_module tf_prefix="${tf_prefix}" name="left" xyz="-0.0024413 0.0886932 0.0298341" rpy="0 0 ${pi/2}"/>
+    <xacro:chassis_module tf_prefix="${tf_prefix}" name="rear" xyz="-0.1581827 -0.0027864 0.0303668" rpy="0 0 ${pi}"/>
+    <xacro:chassis_module tf_prefix="${tf_prefix}" name="right" xyz="-0.0024413 -0.0886932 0.0298341" rpy="0 0 ${-pi/2}"/>
+    <xacro:wheel tf_prefix="${tf_prefix}" name="front_left" xyz="0.1 0.1 0.01535" direction="1" side="1"/>
+    <xacro:wheel tf_prefix="${tf_prefix}" name="front_right" xyz="0.1 -0.1 0.01535" direction="-1" side="-1"/>
+    <xacro:wheel tf_prefix="${tf_prefix}" name="rear_left" xyz="-0.1 0.1 0.01535" direction="-1" side="1"/>
+    <xacro:wheel tf_prefix="${tf_prefix}" name="rear_right" xyz="-0.1 -0.1 0.01535" direction="1" side="-1"/>
     <material name="armor_plastic">
       <color rgba="0.2277128 0.2277128 0.2277128 0.8"/>
@@ -138,7 +104,4 @@
       <color rgba="0.2739087 0.2739087 0.2739087 1.0"/>
     </material>
-    <material name="intelligent_controller">
-      <color rgba="0.8 0.8 0.8 1.0"/>
-    </material>
     <material name="EP_up.001">
       <color rgba="0.0284811 0.0284811 0.0284811 1.0"/>

File: robomaster_description/urdf/camera.urdf.xacro (robot description, xacro)
@@ -1,6 +1,6 @@
 <?xml version="1.0"?>
-<robot xmlns:xacro="http://playerstage.sourceforge.net/gazebo/xmlschema/#xacro" name="robomaster_ep_base">
-  <xacro:macro name="camera" params="">
-    <link name="camera_link">
+<robot xmlns:xacro="http://playerstage.sourceforge.net/gazebo/xmlschema/#xacro">
+  <xacro:macro name="camera" params="tf_prefix='' mount=''">
+    <link name="${tf_prefix}camera_link">
       <inertial>
         <origin xyz="0 0 0" rpy="0 0 0"/>
@@ -16,5 +16,5 @@
       </visual>
     </link>
-    <link name="camera_optical_link">
+    <link name="${tf_prefix}camera_optical_link">
       <inertial>
         <origin xyz="0 0 0" rpy="0 0 0"/>
@@ -23,13 +23,22 @@
       </inertial>
     </link>
-    <joint name="camera_joint" type="fixed">
-      <origin xyz="0.0053865 -0.0195698 0.0473739" rpy="0 1.6898531 0"/>
-      <parent link="arm_2_link"/>
-      <child link="camera_link"/>
-    </joint>
-    <joint name="camera_optical_joint" type="fixed">
+    <xacro:if value="${mount == 'arm'}">
+      <joint name="${tf_prefix}camera_joint" type="fixed">
+        <origin xyz="0.0053865 -0.0195698 0.0473739" rpy="0 1.6898531 0"/>
+        <parent link="${tf_prefix}arm_2_link"/>
+        <child link="${tf_prefix}camera_link"/>
+      </joint>
+    </xacro:if>
+    <xacro:if value="${mount == 'gimbal'}">
+      <joint name="${tf_prefix}camera_joint" type="fixed">
+        <origin xyz="0.0725 0.0 0.119" rpy="0 1.5708 0"/>
+        <parent link="${tf_prefix}gimbal_link"/>
+        <child link="${tf_prefix}camera_link"/>
+      </joint>
+    </xacro:if>
+    <joint name="${tf_prefix}camera_optical_joint" type="fixed">
       <origin xyz="0.002 0.00 0.004" rpy="0.0872663 0 ${-pi/2}"/>
-      <parent link="camera_link"/>
-      <child link="camera_optical_link"/>
+      <parent link="${tf_prefix}camera_link"/>
+      <child link="${tf_prefix}camera_optical_link"/>
     </joint>
     <!-- <joint name="camera_optical_link" type="fixed">
