Commit message: Added meshes. Added S1

File: robomaster_description/urdf/gripper.urdf.xacro (robot description, xacro)
@@ -1,6 +1,6 @@
 <?xml version="1.0"?>
-<robot xmlns:xacro="http://playerstage.sourceforge.net/gazebo/xmlschema/#xacro" name="robomaster_ep_base">
-  <xacro:macro name="gripper" params="">
-        <link name="left_gripper_link_1">
+<robot xmlns:xacro="http://playerstage.sourceforge.net/gazebo/xmlschema/#xacro">
+  <xacro:macro name="gripper" params="tf_prefix=''">
+        <link name="${tf_prefix}left_gripper_link_1">
           <inertial>
             <origin xyz="0 0 0" rpy="0 0 0"/>
@@ -16,5 +16,5 @@
           </visual>
         </link>
-        <link name="left_gripper_link_2">
+        <link name="${tf_prefix}left_gripper_link_2">
           <inertial>
             <origin xyz="0 0 0" rpy="0 0 0"/>
@@ -43,5 +43,5 @@
           </inertial>
         </link> -->
-        <link name="left_gripper_link_4">
+        <link name="${tf_prefix}left_gripper_link_4">
           <inertial>
             <origin xyz="0 0 0" rpy="0 0 0"/>
@@ -63,5 +63,5 @@
           </collision>
         </link>
-        <link name="left_gripper_link_5">
+        <link name="${tf_prefix}left_gripper_link_5">
           <inertial>
             <origin xyz="0 0 0" rpy="0 0 0"/>
@@ -83,5 +83,5 @@
           </collision>
         </link>
-        <link name="left_gripper_link_6">
+        <link name="${tf_prefix}left_gripper_link_6">
           <inertial>
             <origin xyz="0 0 0" rpy="0 0 0"/>
@@ -103,5 +103,5 @@
           </collision>
         </link>
-        <link name="left_gripper_link_7">
+        <link name="${tf_prefix}left_gripper_link_7">
           <inertial>
             <origin xyz="0 0 0" rpy="0 0 0"/>
@@ -123,5 +123,5 @@
           </collision>
         </link>
-        <link name="gripper_link">
+        <link name="${tf_prefix}gripper_link">
           <inertial>
             <origin xyz="0.0326578 -9.78e-05 -0.0327003" rpy="0 0 0"/>
@@ -143,11 +143,11 @@
           </collision>
         </link>
-      <link name="gripper_m_link">
+      <link name="${tf_prefix}gripper_m_link">
       </link>
-      <joint name="gripper_m_joint" type="prismatic">
+      <joint name="${tf_prefix}gripper_m_joint" type="prismatic">
         <limit effort="0" velocity="0" lower="-0.023" upper="0.001"/>
         <origin xyz="0 0 0" rpy="0 0 0"/>
-        <parent link="gripper_link"/>
-        <child link="gripper_m_link"/>
+        <parent link="${tf_prefix}gripper_link"/>
+        <child link="${tf_prefix}gripper_m_link"/>
         <axis xyz="-1 0 0"/>
       </joint>
@@ -159,5 +159,5 @@
           </inertial>
         </link> -->
-        <link name="right_gripper_link_1">
+        <link name="${tf_prefix}right_gripper_link_1">
           <inertial>
             <origin xyz="0 0 0" rpy="0 0 0"/>
@@ -168,10 +168,10 @@
             <origin xyz="-1.52e-05 -8.12e-05 -2.25e-05" rpy="0 0 0"/>
             <geometry>
-              <mesh filename="package://robomaster_description/meshes/EP_cilp_BB_R.001.dae" scale="1.0 1.0 1.0"/>
-            </geometry>
-            <material name="EP_up.001"/>
-          </visual>
-        </link>
-        <link name="right_gripper_link_2">
+              <mesh filename="package://robomaster_description/meshes/right_gripper_1.dae" scale="1.0 1.0 1.0"/>
+            </geometry>
+            <material name="EP_up.001"/>
+          </visual>
+        </link>
+        <link name="${tf_prefix}right_gripper_link_2">
           <inertial>
             <origin xyz="0 0 0" rpy="0 0 0"/>
@@ -200,5 +200,5 @@
           </inertial>
         </link> -->
-        <link name="right_gripper_link_4">
+        <link name="${tf_prefix}right_gripper_link_4">
           <inertial>
             <origin xyz="0 0 0" rpy="0 0 0"/>
@@ -220,5 +220,5 @@
           </collision>
         </link>
-        <link name="right_gripper_link_5">
+        <link name="${tf_prefix}right_gripper_link_5">
           <inertial>
             <origin xyz="0 0 0" rpy="0 0 0"/>
@@ -240,5 +240,5 @@
           </collision>
         </link>
-        <link name="right_gripper_link_6">
+        <link name="${tf_prefix}right_gripper_link_6">
           <inertial>
             <origin xyz="0 0 0" rpy="0 0 0"/>
@@ -260,5 +260,5 @@
           </collision>
         </link>
-        <link name="right_gripper_link_7">
+        <link name="${tf_prefix}right_gripper_link_7">
           <inertial>
             <origin xyz="0 0 0" rpy="0 0 0"/>
@@ -287,15 +287,15 @@
           </inertial>
         </link> -->
-        <joint name="left_gripper_joint_1" type="continuous">
+        <joint name="${tf_prefix}left_gripper_joint_1" type="continuous">
           <origin xyz="0.0163032 0.0212032 -0.0399201" rpy="0 0 0"/>
-          <parent link="gripper_m_link"/>
-          <child link="left_gripper_link_1"/>
-          <axis xyz="0 0 1.0"/>
-          <limit effort="0" velocity="0"/>
-        </joint>
-        <joint name="left_gripper_joint_2" type="continuous">
+          <parent link="${tf_prefix}gripper_m_link"/>
+          <child link="${tf_prefix}left_gripper_link_1"/>
+          <axis xyz="0 0 1.0"/>
+          <limit effort="0" velocity="0"/>
+        </joint>
+        <joint name="${tf_prefix}left_gripper_joint_2" type="continuous">
           <origin xyz="0.0213495 0.0130363 0" rpy="0 0 0"/>
-          <parent link="left_gripper_link_1"/>
-          <child link="left_gripper_link_2"/>
+          <parent link="${tf_prefix}left_gripper_link_1"/>
+          <child link="${tf_prefix}left_gripper_link_2"/>
           <axis xyz="0 0 1.0"/>
           <limit effort="0" velocity="0"/>
@@ -306,22 +306,22 @@
           <child link="left_gripper_link_3_dummy"/>
         </joint> -->
-        <joint name="left_gripper_joint_4" type="continuous">
+        <joint name="${tf_prefix}left_gripper_joint_4" type="continuous">
           <origin xyz="0.00485 0.0204148 -5.8e-06" rpy="0 0 0"/>
-          <parent link="left_gripper_link_2"/>
-          <child link="left_gripper_link_4"/>
-          <axis xyz="0 0 1.0"/>
-          <limit effort="0" velocity="0"/>
-        </joint>
-        <joint name="left_gripper_joint_6" type="continuous">
+          <parent link="${tf_prefix}left_gripper_link_2"/>
+          <child link="${tf_prefix}left_gripper_link_4"/>
+          <axis xyz="0 0 1.0"/>
+          <limit effort="0" velocity="0"/>
+        </joint>
+        <joint name="${tf_prefix}left_gripper_joint_6" type="continuous">
           <origin xyz="0.0051144 -0.0140851 0" rpy="0 0 0"/>
-          <parent link="left_gripper_link_5"/>
-          <child link="left_gripper_link_6"/>
-          <axis xyz="0 0 1.0"/>
-          <limit effort="0" velocity="0"/>
-        </joint>
-        <joint name="left_gripper_joint_7" type="continuous">
+          <parent link="${tf_prefix}left_gripper_link_5"/>
+          <child link="${tf_prefix}left_gripper_link_6"/>
+          <axis xyz="0 0 1.0"/>
+          <limit effort="0" velocity="0"/>
+        </joint>
+        <joint name="${tf_prefix}left_gripper_joint_7" type="continuous">
           <origin xyz="-0.0148823 -0.0168513 0" rpy="0 0 0"/>
-          <parent link="left_gripper_link_6"/>
-          <child link="left_gripper_link_7"/>
+          <parent link="${tf_prefix}left_gripper_link_6"/>
+          <child link="${tf_prefix}left_gripper_link_7"/>
           <axis xyz="0 0 1.0"/>
           <limit effort="0" velocity="0"/>
@@ -332,27 +332,27 @@
           <child link="left_gripper_8_link_dummy"/>
         </joint> -->
-        <joint name="left_gripper_joint_5" type="continuous">
+        <joint name="${tf_prefix}left_gripper_joint_5" type="continuous">
           <origin xyz="0.0385916 0.0103143 1.6e-06" rpy="0 0 0"/>
-          <parent link="left_gripper_link_4"/>
-          <child link="left_gripper_link_5"/>
-          <axis xyz="0 0 1.0"/>
-          <limit effort="0" velocity="0"/>
-        </joint>
-        <joint name="gripper_link" type="fixed">
+          <parent link="${tf_prefix}left_gripper_link_4"/>
+          <child link="${tf_prefix}left_gripper_link_5"/>
+          <axis xyz="0 0 1.0"/>
+          <limit effort="0" velocity="0"/>
+        </joint>
+        <joint name="${tf_prefix}gripper_link" type="fixed">
           <origin xyz="0.0002793 -0.027026 0.0001815" rpy="0 0 0"/>
-          <parent link="endpoint_bracket_link"/>
-          <child link="gripper_link"/>
-        </joint>
-        <joint name="right_gripper_joint_1" type="continuous">
+          <parent link="${tf_prefix}endpoint_bracket_link"/>
+          <child link="${tf_prefix}gripper_link"/>
+        </joint>
+        <joint name="${tf_prefix}right_gripper_joint_1" type="continuous">
           <origin xyz="0.0163034 -0.0209781 -0.0399201" rpy="0 0 0"/>
-          <parent link="gripper_m_link"/>
-          <child link="right_gripper_link_1"/>
-          <axis xyz="0 0 1.0"/>
-          <limit effort="0" velocity="0"/>
-        </joint>
-        <joint name="right_gripper_joint_2" type="continuous">
+          <parent link="${tf_prefix}gripper_m_link"/>
+          <child link="${tf_prefix}right_gripper_link_1"/>
+          <axis xyz="0 0 1.0"/>
+          <limit effort="0" velocity="0"/>
+        </joint>
+        <joint name="${tf_prefix}right_gripper_joint_2" type="continuous">
           <origin xyz="0.0213495 -0.0130363 0" rpy="0 0 0"/>
-          <parent link="right_gripper_link_1"/>
-          <child link="right_gripper_link_2"/>
+          <parent link="${tf_prefix}right_gripper_link_1"/>
+          <child link="${tf_prefix}right_gripper_link_2"/>
           <axis xyz="0 0 1.0"/>
           <limit effort="0" velocity="0"/>
@@ -363,29 +363,29 @@
           <child link="right_gripper_link_3_dummy"/>
         </joint> -->
-        <joint name="right_gripper_joint_4" type="continuous">
+        <joint name="${tf_prefix}right_gripper_joint_4" type="continuous">
           <origin xyz="0.0047151 -0.0208481 -5.8e-06" rpy="0 0 0"/>
-          <parent link="right_gripper_link_2"/>
-          <child link="right_gripper_link_4"/>
-          <axis xyz="0 0 1.0"/>
-          <limit effort="0" velocity="0"/>
-        </joint>
-        <joint name="right_gripper_joint_5" type="continuous">
+          <parent link="${tf_prefix}right_gripper_link_2"/>
+          <child link="${tf_prefix}right_gripper_link_4"/>
+          <axis xyz="0 0 1.0"/>
+          <limit effort="0" velocity="0"/>
+        </joint>
+        <joint name="${tf_prefix}right_gripper_joint_5" type="continuous">
           <origin xyz="0.0385916 -0.0103143 1.6e-06" rpy="0 0 0"/>
-          <parent link="right_gripper_link_4"/>
-          <child link="right_gripper_link_5"/>
-          <axis xyz="0 0 1.0"/>
-          <limit effort="0" velocity="0"/>
-        </joint>
-        <joint name="right_gripper_joint_6" type="continuous">
+          <parent link="${tf_prefix}right_gripper_link_4"/>
+          <child link="${tf_prefix}right_gripper_link_5"/>
+          <axis xyz="0 0 1.0"/>
+          <limit effort="0" velocity="0"/>
+        </joint>
+        <joint name="${tf_prefix}right_gripper_joint_6" type="continuous">
           <origin xyz="0.0059278 0.0133069 0" rpy="0 0 0"/>
-          <parent link="right_gripper_link_5"/>
-          <child link="right_gripper_link_6"/>
-          <axis xyz="0 0 1.0"/>
-          <limit effort="0" velocity="0"/>
-        </joint>
-        <joint name="right_gripper_joint_7" type="continuous">
+          <parent link="${tf_prefix}right_gripper_link_5"/>
+          <child link="${tf_prefix}right_gripper_link_6"/>
+          <axis xyz="0 0 1.0"/>
+          <limit effort="0" velocity="0"/>
+        </joint>
+        <joint name="${tf_prefix}right_gripper_joint_7" type="continuous">
           <origin xyz="-0.0156955 0.0176295 0" rpy="0 0 0"/>
-          <parent link="right_gripper_link_6"/>
-          <child link="right_gripper_link_7"/>
+          <parent link="${tf_prefix}right_gripper_link_6"/>
+          <child link="${tf_prefix}right_gripper_link_7"/>
           <axis xyz="0 0 1.0"/>
           <limit effort="0" velocity="0"/>

File: robomaster_description/urdf/intelligent_controller.urdf.xacro (robot description, xacro)
@@ -1,6 +1,6 @@
 <?xml version="1.0"?>
 <robot xmlns:xacro="http://playerstage.sourceforge.net/gazebo/xmlschema/#xacro">
-  <xacro:macro name="intelligent_controller">
-    <link name="intelligent_controller_link">
+  <xacro:macro name="intelligent_controller" params="tf_prefix='' mount=''">
+    <link name="${tf_prefix}intelligent_controller_link">
       <inertial>
         <origin xyz="0 0 0" rpy="0 0 0"/>
@@ -36,9 +36,21 @@
       </collision>
     </link>
-    <joint name="intelligent_controller_joint" type="fixed">
-      <origin xyz="-0.1348326 0.0024866 0.1329" rpy="0 0 0"/>
-      <parent link="chassis_base_link"/>
-      <child link="intelligent_controller_link"/>
-    </joint>
+    <xacro:if value="${mount == 'extension'}">
+      <joint name="${tf_prefix}intelligent_controller_joint" type="fixed">
+        <origin xyz="-0.1348326 0.0024866 0.1329" rpy="0 0 0"/>
+        <parent link="${tf_prefix}chassis_base_link"/>
+        <child link="${tf_prefix}intelligent_controller_link"/>
+      </joint>
+    </xacro:if>
+    <xacro:if value="${mount == 'gimbal'}">
+      <joint name="${tf_prefix}intelligent_controller_joint" type="fixed">
+        <origin xyz="-0.027 0.0 0.07" rpy="0 0 0"/>
+        <parent link="${tf_prefix}blaster_link"/>
+        <child link="${tf_prefix}intelligent_controller_link"/>
+      </joint>
+    </xacro:if>
+    <material name="intelligent_controller">
+      <color rgba="0.8 0.8 0.8 1.0"/>
+    </material>
   </xacro:macro>
 </robot>

File: robomaster_description/urdf/led.urdf.xacro (robot description, xacro)
@@ -1,6 +1,6 @@
 <?xml version="1.0"?>
-<robot xmlns:xacro="http://playerstage.sourceforge.net/gazebo/xmlschema/#xacro" name="robomaster_ep_base">
-  <xacro:macro name="chassis_module" params="name xyz rpy">
-  <link name="${name}_hit_sensor_link">
+<robot xmlns:xacro="http://playerstage.sourceforge.net/gazebo/xmlschema/#xacro">
+  <xacro:macro name="chassis_module" params="name xyz rpy tf_prefix=''">
+  <link name="${tf_prefix}${name}_hit_sensor_link">
     <inertial>
       <origin xyz="0 0 0" rpy="0 0 0"/>
@@ -16,5 +16,5 @@
     </visual>
   </link>
-  <link name="${name}_led_link">
+  <link name="${tf_prefix}${name}_led_link">
     <inertial>
       <origin xyz="0 0 0" rpy="0 0 0"/>
@@ -30,13 +30,13 @@
     </visual>
   </link>
-  <joint name="${name}_hit_sensor_joint" type="fixed">
+  <joint name="${tf_prefix}${name}_hit_sensor_joint" type="fixed">
     <origin xyz="${xyz}" rpy="${rpy}"/>
-    <parent link="chassis_base_link"/>
-    <child link="${name}_hit_sensor_link"/>
+    <parent link="${tf_prefix}chassis_base_link"/>
+    <child link="${tf_prefix}${name}_hit_sensor_link"/>
   </joint>
-  <joint name="${name}_led_joint" type="fixed">
+  <joint name="${tf_prefix}${name}_led_joint" type="fixed">
     <origin xyz="0.0087428 -0.0012841 3.75e-05" rpy="0 0 0"/>
-    <parent link="${name}_hit_sensor_link"/>
-    <child link="${name}_led_link"/>
+    <parent link="${tf_prefix}${name}_hit_sensor_link"/>
+    <child link="${tf_prefix}${name}_led_link"/>
   </joint>
   </xacro:macro>

File: robomaster_description/urdf/robomaster_ep.urdf.xacro (robot description, xacro)
@@ -1,26 +1,23 @@
 <?xml version="1.0"?>
 <robot name="robomaster_ep" xmlns:xacro="http://playerstage.sourceforge.net/gazebo/xmlschema/#xacro">
+  <xacro:arg name="name" default=""/>
+  <xacro:property name="_name" value="$(arg name)"/>
+  <xacro:if value="${_name != ''}">
+    <xacro:property name="tf_prefix" value="${_name}/"/>
+  </xacro:if>
+  <xacro:if value="${_name == ''}">
+    <xacro:property name="tf_prefix" value=""/>
+  </xacro:if>
   <xacro:include filename="base.urdf.xacro"/>
   <xacro:include filename="arm.urdf.xacro"/>
   <xacro:include filename="camera.urdf.xacro"/>
   <xacro:include filename="gripper.urdf.xacro"/>
-  <xacro:robomaster_ep_base/>
-  <xacro:arm/>
-  <xacro:camera/>
-  <xacro:gripper/>
-<!--
-  <link name="sphere">
-    <visual>
-      <geometry>
-        <sphere radius="1.0"/>
-      </geometry>
-      <material name="wheel_bolt">
-        <color rgba="0.6 0.2 0.0 1.0"/>
-      </material>
-    </visual>
-  </link>
-  <joint name="sphere_joint" type="fixed">
-    <parent link="base_link"/>
-    <child link="sphere"/>
-  </joint> -->
+  <xacro:include filename="intelligent_controller.urdf.xacro"/>
+  <xacro:include filename="extension.urdf.xacro"/>
+  <xacro:base tf_prefix="${tf_prefix}"/>
+  <xacro:extension tf_prefix="${tf_prefix}" use_rear_extension="true"/>
+  <xacro:intelligent_controller tf_prefix="${tf_prefix}" mount="extension"/>
+  <xacro:arm tf_prefix="${tf_prefix}"/>
+  <xacro:camera tf_prefix="${tf_prefix}" mount="arm"/>
+  <xacro:gripper tf_prefix="${tf_prefix}"/>
 </robot>

File: robomaster_description/urdf/wheel.urdf.xacro (robot description, xacro)
@@ -1,6 +1,6 @@
 <?xml version="1.0"?>
-<robot xmlns:xacro="http://playerstage.sourceforge.net/gazebo/xmlschema/#xacro" name="robomaster_ep_base">
-  <xacro:macro name="wheel" params="name xyz direction side">
-    <link name="${name}_wheel_link">
+<robot xmlns:xacro="http://playerstage.sourceforge.net/gazebo/xmlschema/#xacro">
+  <xacro:macro name="wheel" params="name xyz direction side tf_prefix=''">
+    <link name="${tf_prefix}${name}_wheel_link">
       <inertial>
         <origin xyz="-0.0002104 5.31e-05 -0.0004148" rpy="0 0 0"/>
@@ -34,8 +34,8 @@
       </collision>
     </link>
-    <joint name="${name}_wheel_joint" type="continuous">
+    <joint name="${tf_prefix}${name}_wheel_joint" type="continuous">
       <origin xyz="${xyz}" rpy="0 0 0"/>
-      <parent link="chassis_base_link"/>
-      <child link="${name}_wheel_link"/>
+      <parent link="${tf_prefix}chassis_base_link"/>
+      <child link="${tf_prefix}${name}_wheel_link"/>
       <axis xyz="0 1.0 0"/>
       <limit effort="0" velocity="0"/>
