Commit message: Large commit with servo [actions], gimbal, blaster and correct tf frames

File: robomaster_description/urdf/camera.urdf.xacro (robot description, xacro)
@@ -32,6 +32,6 @@
     <xacro:if value="${mount == 'gimbal'}">
       <joint name="${tf_prefix}camera_joint" type="fixed">
-        <origin xyz="0.0725 0.0 0.119" rpy="0 1.5708 0"/>
-        <parent link="${tf_prefix}gimbal_link"/>
+        <origin xyz="0.0728 0.0 0.0315" rpy="0 1.5708 0"/>
+        <parent link="${tf_prefix}blaster_link"/>
         <child link="${tf_prefix}camera_link"/>
       </joint>

File: robomaster_description/urdf/gimbal.urdf.xacro (robot description, xacro)
@@ -82,12 +82,117 @@
         <material name="led_off" />
       </visual>
+      <visual name="gimbal_left_led_0">
+        <origin xyz="-0.02365 0 -0.01734" rpy="0 0 0"/>
+        <geometry>
+          <mesh filename="package://robomaster_description/meshes/gimbal_left_led_0.dae" scale="1.0 1.0 1.0"/>
+        </geometry>
+        <material name="led_off"/>
+      </visual>
+      <visual name="gimbal_left_led_1">
+        <origin xyz="-0.00837 0 -0.02777" rpy="0 0 0"/>
+        <geometry>
+          <mesh filename="package://robomaster_description/meshes/gimbal_left_led_1.dae" scale="1.0 1.0 1.0"/>
+        </geometry>
+        <material name="led_off"/>
+      </visual>
+      <visual name="gimbal_left_led_2">
+        <origin xyz="0.01027 0 -0.02687" rpy="0 0 0"/>
+        <geometry>
+          <mesh filename="package://robomaster_description/meshes/gimbal_left_led_2.dae" scale="1.0 1.0 1.0"/>
+        </geometry>
+        <material name="led_off"/>
+      </visual>
+      <visual name="gimbal_left_led_3">
+        <origin xyz="0.02428 0 -0.01501" rpy="0 0 0"/>
+        <geometry>
+          <mesh filename="package://robomaster_description/meshes/gimbal_left_led_3.dae" scale="1.0 1.0 1.0"/>
+        </geometry>
+        <material name="led_off"/>
+      </visual>
+      <visual name="gimbal_left_led_4">
+        <origin xyz="0.02289 -4e-05 0.01672" rpy="0 0 0"/>
+        <geometry>
+          <mesh filename="package://robomaster_description/meshes/gimbal_left_led_4.dae" scale="1.0 1.0 1.0"/>
+        </geometry>
+        <material name="led_off"/>
+      </visual>
+      <visual name="gimbal_left_led_5">
+        <origin xyz="0.00874 0 0.02703" rpy="0 0 0"/>
+        <geometry>
+          <mesh filename="package://robomaster_description/meshes/gimbal_left_led_5.dae" scale="1.0 1.0 1.0"/>
+        </geometry>
+        <material name="led_off"/>
+      </visual>
+      <visual name="gimbal_left_led_6">
+        <origin xyz="-0.00951 1e-05 0.02709" rpy="0 0 0"/>
+        <geometry>
+          <mesh filename="package://robomaster_description/meshes/gimbal_left_led_6.dae" scale="1.0 1.0 1.0"/>
+        </geometry>
+        <material name="led_off"/>
+      </visual>
+      <visual name="gimbal_left_led_7">
+        <origin xyz="-0.02463 0 0.01615" rpy="0 0 0"/>
+        <geometry>
+          <mesh filename="package://robomaster_description/meshes/gimbal_left_led_7.dae" scale="1.0 1.0 1.0"/>
+        </geometry>
+        <material name="led_off"/>
+      </visual>
     </link>
     <link name="${tf_prefix}gimbal_right_led_link">
-      <visual name="gimbal_right_led">
-        <origin xyz="-0.02364 -9e-05 -0.01734" rpy="0 0 0" />
-        <geometry>
-          <mesh filename="package://robomaster_description/meshes/gimbal_right_led.dae" scale="1.0 1.0 1.0" />
-        </geometry>
-        <material name="led_off" />
+      <visual name="gimbal_right_led_0">
+        <origin xyz="-0.02364 -9e-05 -0.01734" rpy="0 0 0"/>
+        <geometry>
+          <mesh filename="package://robomaster_description/meshes/gimbal_right_led_0.dae" scale="1.0 1.0 1.0"/>
+        </geometry>
+        <material name="led_off"/>
+      </visual>
+      <visual name="gimbal_right_led_1">
+        <origin xyz="-0.00837 -0.00011 -0.02778" rpy="0 0 0"/>
+        <geometry>
+          <mesh filename="package://robomaster_description/meshes/gimbal_right_led_1.dae" scale="1.0 1.0 1.0"/>
+        </geometry>
+        <material name="led_off"/>
+      </visual>
+      <visual name="gimbal_right_led_2">
+        <origin xyz="0.01027 -0.00011 -0.02687" rpy="0 0 0"/>
+        <geometry>
+          <mesh filename="package://robomaster_description/meshes/gimbal_right_led_2.dae" scale="1.0 1.0 1.0"/>
+        </geometry>
+        <material name="led_off"/>
+      </visual>
+      <visual name="gimbal_right_led_3">
+        <origin xyz="0.02428 -0.00011 -0.01501" rpy="0 0 0"/>
+        <geometry>
+          <mesh filename="package://robomaster_description/meshes/gimbal_right_led_3.dae" scale="1.0 1.0 1.0"/>
+        </geometry>
+        <material name="led_off"/>
+      </visual>
+      <visual name="gimbal_right_led_4">
+        <origin xyz="0.0229 0.00017 0.01671" rpy="0 0 0"/>
+        <geometry>
+          <mesh filename="package://robomaster_description/meshes/gimbal_right_led_4.dae" scale="1.0 1.0 1.0"/>
+        </geometry>
+        <material name="led_off"/>
+      </visual>
+      <visual name="gimbal_right_led_5">
+        <origin xyz="0.00874 8e-05 0.02709" rpy="0 0 0"/>
+        <geometry>
+          <mesh filename="package://robomaster_description/meshes/gimbal_right_led_5.dae" scale="1.0 1.0 1.0"/>
+        </geometry>
+        <material name="led_off"/>
+      </visual>
+      <visual name="gimbal_right_led_6">
+        <origin xyz="-0.00957 8e-05 0.02706" rpy="0 0 0"/>
+        <geometry>
+          <mesh filename="package://robomaster_description/meshes/gimbal_right_led_6.dae" scale="1.0 1.0 1.0"/>
+        </geometry>
+        <material name="led_off"/>
+      </visual>
+      <visual name="gimbal_right_led_7">
+        <origin xyz="-0.02463 8e-05 0.01615" rpy="0 0 0"/>
+        <geometry>
+          <mesh filename="package://robomaster_description/meshes/gimbal_right_led7.dae" scale="1.0 1.0 1.0"/>
+        </geometry>
+        <material name="led_off"/>
       </visual>
     </link>
@@ -164,5 +269,5 @@
       <axis xyz="0 1.0 0"/>
       <!-- [-25, +30] degrees -->
-      <limit effort="0" velocity="0" lower="-0.4363" upper="0.5236"/>
+      <limit effort="0" velocity="0" lower="-0.5236" upper="0.4363"/>
     </joint>
     <joint name="${tf_prefix}gimbal_left_led_joint" type="fixed">

Commit message: Updated

File: robomaster_description/urdf/camera.urdf.xacro (robot description, xacro)
@@ -38,5 +38,7 @@
     </xacro:if>
     <joint name="${tf_prefix}camera_optical_joint" type="fixed">
-      <origin xyz="0.002 0.00 0.004" rpy="0.0872663 0 ${-pi/2}"/>
+      <!-- <origin xyz="0.002 0.00 0.004" rpy="0.0872663 0 ${-pi/2}"/> -->
+      <!-- <origin xyz="0.002 0.00 0.004" rpy="0.0072663 0 ${-pi/2}"/> -->
+      <origin xyz="0.002 0.00 0.004" rpy="0.041623 0 ${-pi/2}"/>
       <parent link="${tf_prefix}camera_link"/>
       <child link="${tf_prefix}camera_optical_link"/>

File: robomaster_description/urdf/gripper.urdf.xacro (robot description, xacro)
@@ -144,4 +144,6 @@
         </link>
       <link name="${tf_prefix}gripper_m_link">
+      </link>
+      <link name="${tf_prefix}gripper_t_link">
       </link>
       <joint name="${tf_prefix}gripper_m_joint" type="prismatic">
@@ -396,4 +398,9 @@
           <child link="right_gripper_link_8_dummy"/>
         </joint> -->
+        <joint name="${tf_prefix}gripper_joint_t" type="fixed">
+          <origin xyz="0.124 0 -0.039" rpy="0 0 0"/>
+          <parent link="${tf_prefix}gripper_link"/>
+          <child link="${tf_prefix}gripper_t_link"/>
+        </joint>
   </xacro:macro>
 </robot>

File: robomaster_description/urdf/robomaster_ep.urdf.xacro (robot description, xacro)
@@ -15,4 +15,5 @@
   <xacro:include filename="intelligent_controller.urdf.xacro"/>
   <xacro:include filename="extension.urdf.xacro"/>
+  <xacro:include filename="tof.urdf.xacro"/>
   <xacro:base tf_prefix="${tf_prefix}"/>
   <xacro:extension tf_prefix="${tf_prefix}" use_rear_extension="true"/>
@@ -21,3 +22,7 @@
   <xacro:camera tf_prefix="${tf_prefix}" mount="arm"/>
   <xacro:gripper tf_prefix="${tf_prefix}"/>
+  <xacro:add_tof index="0" tf_prefix="${tf_prefix}"/>
+  <xacro:add_tof index="1" tf_prefix="${tf_prefix}"/>
+  <xacro:add_tof index="2" tf_prefix="${tf_prefix}"/>
+  <xacro:add_tof index="3" tf_prefix="${tf_prefix}"/>
 </robot>

File: robomaster_description/urdf/robomaster_s1.urdf.xacro (robot description, xacro)
@@ -13,7 +13,12 @@
   <xacro:include filename="camera.urdf.xacro"/>
   <xacro:include filename="intelligent_controller.urdf.xacro"/>
+  <xacro:include filename="tof.urdf.xacro"/>
   <xacro:base tf_prefix="${tf_prefix}"/>
   <xacro:gimbal tf_prefix="${tf_prefix}"/>
   <xacro:camera tf_prefix="${tf_prefix}" mount="gimbal"/>
   <xacro:intelligent_controller tf_prefix="${tf_prefix}" mount="gimbal"/>
+  <xacro:add_tof index="0" tf_prefix="${tf_prefix}"/>
+  <xacro:add_tof index="1" tf_prefix="${tf_prefix}"/>
+  <xacro:add_tof index="2" tf_prefix="${tf_prefix}"/>
+  <xacro:add_tof index="3" tf_prefix="${tf_prefix}"/>
 </robot>

Commit message: Added arm servo index and camera yaw parameters

File: robomaster_description/urdf/camera.urdf.xacro (robot description, xacro)
@@ -1,5 +1,5 @@
 <?xml version="1.0"?>
 <robot xmlns:xacro="http://playerstage.sourceforge.net/gazebo/xmlschema/#xacro">
-  <xacro:macro name="camera" params="tf_prefix='' mount=''">
+  <xacro:macro name="camera" params="tf_prefix='' mount='' camera_yaw=0.0">
     <link name="${tf_prefix}camera_link">
       <inertial>
@@ -25,5 +25,5 @@
     <xacro:if value="${mount == 'arm'}">
       <joint name="${tf_prefix}camera_joint" type="fixed">
-        <origin xyz="0.0053865 -0.0195698 0.0473739" rpy="0 1.6898531 0"/>
+        <origin xyz="0.0053865 -0.0195698 0.0473739" rpy="0 1.6898531 ${camera_yaw}"/>
         <parent link="${tf_prefix}arm_2_link"/>
         <child link="${tf_prefix}camera_link"/>
